File: ngin-link-hw.kicad_sch (KiCad schematic)
At the start: 0 parts

Commit message: feat: add hierarchical schematic and isolated USB/CAN power architecture
Schematic (sch/):
- Introduce 2-level hierarchy: root (title + index) -> block diagram
  (sch/01_block_diagram.kicad_sch) -> 4 functional sheets
  (10_usb, 20_power, 30_mcu, 40_can).
- Functional sheets are placeholder block diagrams with rectangle + text
  annotations; components and wires to be added in the KiCad editor.
- LEDs (PB0/PB1) and SWD (Tag-Connect) live inside the 30_mcu sheet.

Hardware architecture (README.md, AGENTS.md):
- Galvanic isolation between USB VBUS and CAN bus using B0505S isolated
  DC-DC (5V/5V, 1W) on the power path and ADUM1201 dual-channel digital
  isolator on CAN TX/RX.
- Power tree split into USB side (GND_USB, +3V3_USB) and CAN side
  (GND_ISO, VISO_5V, +3V3_CAN); MCU on USB side, SN65HVD230 on CAN side.

Tooling:
- Ignore *.kicad_prl (per-user UI state, regenerated by KiCad on open).
- Drop one-off Python bootstrap/cleanup scripts; .kicad_sch files are
  the source of truth.
Other:
- added sheet Block Diagram (sch/01_block_diagram.kicad_sch)
- note added: "#"
- note added: "${ISSUE_DATE}"
- note added: "${REVISION}"
- note added: "/"
- note added: "1"
- note added: "2"
- note added: "2026-06-28"
- note added: "3"
- note added: "4"
- note added: "5"
- note added: "6"
- note added: "A"
- note added: "AP2112K-3.3 LDO + filtering"
- note added: "ARR"
- note added: "Author"
- note added: "Author:"
- note added: "Block diagram (top level)"
- note added: "CERN-OHL-S 2.0"
- note added: "Click the sheet block to navigate to the block diagram (Sheet 2)."
- note added: "Company:"
- note added: "Date"
- note added: "Date:"
- note added: "Description"
- note added: "File"
- note added: "INDEX"
- note added: "Initial release - hierarchical structure"
- note added: "KiCad 10.x hierarchical schematic. See README.md for details."
- note added: "License:"
- note added: "NGIN-LINK"
- note added: "Ngin performance"
- note added: "Ngin-link USB to CAN dongle"
- note added: "PROJECT INFORMATION"
- note added: "Project:"
- note added: "Prototype"
- note added: "REVISION HISTORY"
- note added: "Rev"
- note added: "Revision:"
- note added: "SN65HVD230 + TVS + termination + isolation"
- note added: "STM32F446RET6 + crystal + reset"
- note added: "STM32F446RET6 | SN65HVD230 | USB 2.0 FS"
- note added: "Sheet"
- note added: "Status:"
- note added: "Title, index, project info"
- note added: "Title:"
- note added: "USB-C + ESD + CC pull-downs"
- note added: "USB-C to CAN FD Bridge Dongle"
- note added: "ngin-link-hw"
- note added: "sch/01_block_diagram.kicad_sch"
- note added: "sch/10_usb.kicad_sch"
- note added: "sch/20_power.kicad_sch"
- note added: "sch/30_mcu.kicad_sch"
- note added: "sch/40_can.kicad_sch"
- company: (none) -> Ngin performance
- title: (none) -> Ngin-link USB to CAN dongle

Commit message: Update ngin-link-hw.kicad_sch
Se cambio la denominación del estatus del esquemático.
Other:
- note added: "Draft"
- note removed: "Author"
- note removed: "Prototype"
